File: Wiring/LPS-1 Wiring/LPS-1 Wiring.kicad_pcb (KiCad board)
At the start: 32 copper layers, 26 parts, among them J1 Block_Connector_01_b, J10 Block_Connector_01_b, J101 Block_Connector_01_b, J102 Block_Connector_01_b, J11 Block_Connector_01_b, J12 Block_Connector_01_b, J13 Block_Connector_01_b, J2 Block_Connector_01_b, J3 Block_Connector_01_b, J4 Block_Connector_01_b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

Commit message: Panel wiring update
Parts:
- added J13: Block_Connector_01_b, Wiring:Degson_01_PC2.5-01P-11-00AH-1_5.2, F.Cu at (635.3, 442.5)
- moved J14 3.91 mm to (641.4, 442.2)
- moved J101 0.40 mm to (649.2, 442.2)
- moved J102 0.20 mm to (655.2, 442.2)
- renumbered J13 to J14
Connections:
- FB1 pad 2: /LPS-12V -> /LPS-12V_1
- J12 pad 1: Net-(LPS1-Pin_1) -> /LPS-12V
- J12 pad 2: /LPS-12V -> /LPS-12V_3
- LPS1 pad 1: Net-(LPS1-Pin_1) -> /LPS-12V
- SW3 pad 5: unconnected-(SW3B-11-Pad5) -> /LPS-12V_2
- SW3 pad 6: unconnected-(SW3B-12-Pad6) -> /LPS-12V_3
Routing:
- net /LPS-12V_1: track 0.00 -> 459.2 mm
- net Net-(LPS1-Pin_1): track 299.6 -> 0.00 mm
- net /LPS-12V: track 360.9 -> 299.1 mm
- net /LPS-12V_3: track 0.00 -> 54.8 mm
- net /LPS-12V_2: track 0.00 -> 46.9 mm
- net /SOL_CHRG-: track 226.1 -> 196.7 mm
- net /SOL_CHRG+: track 212.4 -> 188.7 mm
- net Net-(SC1-Pin_2): track 201.3 -> 181.8 mm
- net Net-(SC1-Pin_1): track 188.8 -> 175.7 mm
- net /PWR-COMM-B: track 241.1 -> 235.1 mm
- net /PWR-COMM-A: track 83.4 -> 87.7 mm
Other:
- board text added: "14.1"
- board text added: "14.2"
