File: pcb/lps-1.kicad_sch (KiCad schematic)
At the start: 26 parts, among them J15 PWR, J4 A_INA219, J5 XBEE, J6 DEV, U1 L7805, U2 ATMega1608_32, U3 TC1262-33

Commit message: Update and sync
Changed lines of the file:
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@@
 (kicad_sch
-	(version 20231120)
+	(version 20250114)
 	(generator "eeschema")
-	(generator_version "8.0")
+	(generator_version "9.0")
 	(paper "A3")
 	(title_block
@@
 		(rev "1.2.1")
 	)
+	(text "DIN\nDOUT\n~{SLEEP_REQ}\n~{RESET}\n3V3\nGND"
+		(exclude_from_sim no)
+		(at 78.232 189.738 0)
+		(effects
+			(font
+				(size 1.27 1.27)
+			)
+			(justify right bottom)
+		)
+	)
 	(junction
 		(at 99.06 64.77)
@@
 			"dASRBwA6gsgDAB1B5AGAjiDyAEBHEHkAoCOIPADQEUQeAOgIIg8AdASRBwA6gsgDAB1B5AGAjiDy"
 			"AEBHEHkAoCOIPADQEUQeAOgIIg8AdASRBwA6gsgDAB1B5AGAjiDyAEBHEHkAoCOIPADQEUQeAOgI"
-			"Ig8AdASRBwA68j9Gwq8M7Z+K4QAAAABJRU5ErkJggg=="
-		)
-	)
-	(text "DIN\nDOUT\n~{SLEEP_REQ}\n~{RESET}\n3V3\nGND"
-		(exclude_from_sim no)
-		(at 78.232 189.738 0)
-		(effects
-			(font
-				(size 1.27 1.27)
-			)
-			(justify right bottom)
+			"Ig8AdASRBwA68j9Gwq8M7Z+K4QAAAABJRU5ErkJgggAAAAAAAAAAAAAAAAAAAAAAAAAAAAAAAAAA"
+			"AAAAAAAAAAAAAAAAAAAAAAAAAAAAAAAAAAAAAAAAAAAAAAAAAAAAAAAAAAAAAAAAAAAAAAAAAAAA"
+			"AAAAAAAAAAAAAAAAAAAAAAAAAAAAAAAAAAAAAAAAAAAAAAAAAAAAAAAAAAAAAAAAAAAAAAAAAAAA"
+			"AAAAAAAAAAAAAAAAAAAAAAAAAAAAAAAAAAAAAAAAAAAAAAAAAAAAAAAAAAAAAAAAAAAAAAAAAAAA"
+			"AAAAAAAAAAAAAAAAAAAAAAAAAAAAAAAAAAAAAAAAAAAAAAAAAAAAAAAAAAAAAAAAAAAAAAAAAAAA"
+			"AAAAAAAAAAAAAAAAAAAAAAAAAAAAAAAAAAAAAAAAAAAAAAAAAAAAAAAAAAAAAAAAAAAAAAAAAAAA"
+			"AAAAAAAAAAAAAAAAAAAAAAAAAAAAAAAAAAAAAAAAAAAAAAAAAAAAAAAAAAAAAAAAAAAAAAAAAAAA"
+			"AAAAAAAAAAAAAAAAAAAAAAAAAAAAAAAAAAAAAAAAAAAAAAAAAAAAAAAAAAAAAAAAAAAAAAAAAAAA"
+			"AAAAAAAAAAAAAAAAAAAAAAAAAAAAAAAAAAAAAAAAAAAAAAAAAAAAAAAAAAAAAAAAAAAAAAAAAAAA"
+			"AAAAAAAAAAAAAAAAAAAAAAAAAAAAAAAAAAAAAAAAAAAAAAAAAAAAAAAAAAAAAAAAAAAAAAAAAAAA"
+			"AAAAAAAAAAAAAAAAAAAAAAAAAAAAAAAAAAAAAAAAAAAAAAAAAAAAAAAAAAAAAAAAAAAAAAAAAAAA"
+			"AAAAAAAAAAAAAAAAAAAAAAAAAAAAAAAAAAAAAAAAAAAAAAAAAAAAAAAAAAAAAAAAAAAAAAAAAAAA"
+			"AAAAAAAAAAAAAAAAAAAAAAAAAAAAAAAAAAAAAAAAAAAAAAAAAAAAAAAAAAAAAAAAAAAAAAAAAAAA"
+			"AAAAAAAAAAAAAAAAAAAAAAAAAAAAAAAAAAAAAAAAAAAAAAAAAAAAAAAAAAAAAAAAAAAAAAAAAAAA"
+			"AAAAAAAAAAAAAAAAAAAAAAAAAAAAAAAAAAAAAAAAAAAAAAAAAAAAAAAAAAAAAAAAAAAAAAAAAAAA"
+			"AAAAAAAAAAAAAAAAAAAAAAAAAAAAAAAAAAAAAAAAAAAAAAAAAAAAAAAAAAAAAAAAAAAAAAAAAAAA"
+			"AAAAAAAAAAAAAAAAAAAAAAAAAAAAAAAAAAAAAAAAAAAAAAAAAAAAAAAAAAAAAAAAAAAAAAAAAAAA"
+			"AAAAAAAAAAAAAAAAAAAAAAAAAAAAAAAAAAAAAAAAAAAAAAAAAAAAAAAAAAAAAAAAAAAAAAAAAAAA"
+			"AAAAAAAAAAAAAAAAAAAAAAAAAAAAAAAAAAAAAAAAAA=="
 		)
 	)
 	(label "SCK"
 		(at 306.07 162.56 180)
-		(fields_autoplaced yes)
 		(effects
 			(font
@@
 	(label "RxD0"
 		(at 93.98 180.34 180)
-		(fields_autoplaced yes)
 		(effects
 			(font
@@
 	(label "RxD0"
 		(at 306.07 160.02 180)
-		(fields_autoplaced yes)
 		(effects
 			(font
@@
 	(label "UPDI"
 		(at 198.12 147.32 0)
-		(fields_autoplaced yes)
 		(effects
 			(font
@@
 	(label "SDA"
 		(at 93.98 162.56 180)
-		(fields_autoplaced yes)
 		(effects
 			(font
@@
 	(label "PD5"
 		(at 306.07 195.58 180)
-		(fields_autoplaced yes)
 		(effects
 			(font
@@
 	(label "MODEM_RESET"
 		(at 101.6 185.42 180)
-		(fields_autoplaced yes)
 		(effects
 			(font
@@
 	(label "DOUT"
 		(at 96.52 218.44 180)
-		(fields_autoplaced yes)
 		(effects
 			(font
@@
 	(label "SS"
 		(at 306.07 165.1 180)
-		(fields_autoplaced yes)
 		(effects
 			(font
@@
 	(label "TxD0"
 		(at 93.98 177.8 180)
-		(fields_autoplaced yes)
 		(effects
 			(font
@@
 	(label "SCL"
 		(at 306.07 146.05 180)
-		(fields_autoplaced yes)
 		(effects
 			(font
@@
 	(label "PD3"
 		(at 306.07 190.5 180)
-		(fields_autoplaced yes)
 		(effects
 			(font
@@
 	(label "MODEM_SLEEP"
 		(at 101.6 182.88 180)
-		(fields_autoplaced yes)
 		(effects
 			(font
@@
 	(label "TxD0"
 		(at 306.07 157.48 180)
-		(fields_autoplaced yes)
 		(effects
 			(font
@@
 	(label "PF5"
 		(at 306.07 220.98 180)
-		(fields_autoplaced yes)
 		(effects
 			(font
@@
 	(label "PF3"
 		(at 306.07 215.9 180)
-		(fields_autoplaced yes)
 		(effects
 			(font
@@
 	(label "~{RESET}"
 		(at 181.61 140.97 0)
-		(fields_autoplaced yes)
 		(effects
 			(font
@@
 	(label "PC2"
 		(at 306.07 177.8 180)
-		(fields_autoplaced yes)
 		(effects
 			(font
@@
 	(label "PF1"
 		(at 306.07 210.82 180)
-		(fields_autoplaced yes)
 		(effects
 			(font
@@
 	(label "PD7"
 		(at 306.07 200.66 180)
-		(fields_autoplaced yes)
 		(effects
 			(font
@@
 	(label "DIN"
 		(at 306.07 175.26 180)
-		(fields_autoplaced yes)
 		(effects
 			(font
@@
 	(label "MODEM_RESET"
 		(at 306.07 182.88 180)
-		(fields_autoplaced yes)
 		(effects
 			(font
@@
 	(label "PF0"
 		(at 306.07 208.28 180)
-		(fields_autoplaced yes)
 		(effects
 			(font
@@
 	(label "PC3"
 		(at 306.07 180.34 180)
-		(fields_autoplaced yes)
 		(effects
 			(font
@@
 	(label "12VIN"
 		(at 92.71 124.46 180)
-		(fields_autoplaced yes)
 		(effects
 			(font
@@
 	(label "PA1"
 		(at 306.07 153.67 180)
-		(fields_autoplaced yes)
 		(effects
 			(font
@@
 	(label "12VIN"
 		(at 24.13 50.8 0)
-		(fields_autoplaced yes)
 		(effects
 			(font
@@
 	(label "DOUT"
 		(at 306.07 172.72 180)
-		(fields_autoplaced yes)
 		(effects
 			(font
@@
 	(label "PD4"
 		(at 306.07 193.04 180)
-		(fields_autoplaced yes)
 		(effects
 			(font
@@
 	(label "DIN"
 		(at 96.52 213.36 180)
-		(fields_autoplaced yes)
 		(effects
 			(font
@@
 	(label "SDA"
 		(at 306.07 143.51 180)
-		(fields_autoplaced yes)
 		(effects
 			(font
@@
 	(label "PF2"
 		(at 306.07 213.36 180)
-		(fields_autoplaced yes)
 		(effects
 			(font
@@
 	(label "PD6"
 		(at 306.07 198.12 180)
-		(fields_autoplaced yes)
 		(effects
 			(font
@@
 	(label "SCL"
 		(at 93.98 160.02 180)
-		(fields_autoplaced yes)
 		(effects
 			(font
@@
 	(label "PA0"
 		(at 306.07 151.13 180)
-		(fields_autoplaced yes)
 		(effects
 			(font
@@
 	(label "MODEM_SLEEP"
 		(at 306.07 185.42 180)
-		(fields_autoplaced yes)
 		(effects
 			(font
@@
 	(label "UPDI"
 		(at 96.52 208.28 180)
-		(fields_autoplaced yes)
 		(effects
 			(font
@@
 	(label "PD2"
 		(at 306.07 187.96 180)
-		(fields_autoplaced yes)
 		(effects
 			(font
@@
 	(label "PF4"
 		(at 306.07 218.44 180)
-		(fields_autoplaced yes)
 		(effects
 			(font
@@
 		)
 	)
+	(embedded_fonts no)
 )

Commit message: Local update
Parts:
- H3, H4, JP1, Lg1, Lg2, Lg3: now left out of the parts list
Changed lines of the file:
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@@
 		(body_style 1)
 		(exclude_from_sim no)
-		(in_bom yes)
+		(in_bom no)
 		(on_board yes)
 		(in_pos_files yes)
@@
 			)
 		)
+		(property "MPN" ""
+			(at 307.34 100.33 0)
+			(hide yes)
+			(show_name no)
+			(do_not_autoplace no)
+			(effects
+				(font
+					(size 1.27 1.27)
+				)
+			)
+		)
+		(property "Link" ""
+			(at 307.34 100.33 0)
+			(hide yes)
+			(show_name no)
+			(do_not_autoplace no)
+			(effects
+				(font
+					(size 1.27 1.27)
+				)
+			)
+		)
+		(property "Comp_Name" ""
+			(at 307.34 100.33 0)
+			(show_name no)
+			(do_not_autoplace no)
+			(effects
+				(font
+					(size 1.27 1.27)
+				)
+			)
+		)
 		(instances
 			(project "lps-1"
@@
 		(body_style 1)
 		(exclude_from_sim no)
-		(in_bom yes)
+		(in_bom no)
 		(on_board yes)
 		(in_pos_files yes)
@@
 			)
 		)
+		(property "MPN" ""
+			(at 369.57 93.98 0)
+			(hide yes)
+			(show_name no)
+			(do_not_autoplace no)
+			(effects
+				(font
+					(size 1.27 1.27)
+				)
+			)
+		)
+		(property "Link" ""
+			(at 369.57 93.98 0)
+			(hide yes)
+			(show_name no)
+			(do_not_autoplace no)
+			(effects
+				(font
+					(size 1.27 1.27)
+				)
+			)
+		)
+		(property "Comp_Name" ""
+			(at 369.57 93.98 0)
+			(show_name no)
+			(do_not_autoplace no)
+			(effects
+				(font
+					(size 1.27 1.27)
+				)
+			)
+		)
 		(instances
 			(project "lps-1"
@@
 		(body_style 1)
 		(exclude_from_sim no)
-		(in_bom yes)
+		(in_bom no)
 		(on_board yes)
 		(in_pos_files yes)
@@
 			)
 		)
+		(property "MPN" ""
+			(at 168.91 57.15 0)
+			(hide yes)
+			(show_name no)
+			(do_not_autoplace no)
+			(effects
+				(font
+					(size 1.27 1.27)
+				)
+			)
+		)
+		(property "Link" ""
+			(at 168.91 57.15 0)
+			(hide yes)
+			(show_name no)
+			(do_not_autoplace no)
+			(effects
+				(font
+					(size 1.27 1.27)
+				)
+			)
+		)
+		(property "Comp_Name" ""
+			(at 168.91 57.15 0)
+			(show_name no)
+			(do_not_autoplace no)
+			(effects
+				(font
+					(size 1.27 1.27)
+				)
+			)
+		)
 		(pin "1"
 		)
@@
 		(body_style 1)
 		(exclude_from_sim no)
-		(in_bom yes)
+		(in_bom no)
 		(on_board yes)
 		(in_pos_files yes)
@@
 			)
 		)
+		(property "MPN" ""
+			(at 307.34 93.98 0)
+			(hide yes)
+			(show_name no)
+			(do_not_autoplace no)
+			(effects
+				(font
+					(size 1.27 1.27)
+				)
+			)
+		)
+		(property "Link" ""
+			(at 307.34 93.98 0)
+			(hide yes)
+			(show_name no)
+			(do_not_autoplace no)
+			(effects
+				(font
+					(size 1.27 1.27)
+				)
+			)
+		)
+		(property "Comp_Name" ""
+			(at 307.34 93.98 0)
+			(show_name no)
+			(do_not_autoplace no)
+			(effects
+				(font
+					(size 1.27 1.27)
+				)
+			)
+		)
 		(instances
 			(project "lps-1"
@@
 		(body_style 1)
 		(exclude_from_sim no)
-		(in_bom yes)
+		(in_bom no)
 		(on_board yes)
 		(in_pos_files yes)
@@
 			)
 		)
+		(property "MPN" ""
+			(at 346.71 93.98 0)
+			(hide yes)
+			(show_name no)
+			(do_not_autoplace no)
+			(effects
+				(font
+					(size 1.27 1.27)
+				)
+			)
+		)
+		(property "Link" ""
+			(at 346.71 93.98 0)
+			(hide yes)
+			(show_name no)
+			(do_not_autoplace no)
+			(effects
+				(font
+					(size 1.27 1.27)
+				)
+			)
+		)
+		(property "Comp_Name" ""
+			(at 346.71 93.98 0)
+			(show_name no)
+			(do_not_autoplace no)
+			(effects
+				(font
+					(size 1.27 1.27)
+				)
+			)
+		)
 		(instances
 			(project "lps-1"
@@
 		(body_style 1)
 		(exclude_from_sim no)
-		(in_bom yes)
+		(in_bom no)
 		(on_board yes)
 		(in_pos_files yes)
@@
 			(show_name no)
 			(do_not_autoplace no)
+			(effects
+				(font
+					(size 1.27 1.27)
+				)
+			)
+		)
+		(property "MPN" ""
+			(at 358.14 93.98 0)
+			(hide yes)
+			(show_name no)
+			(do_not_autoplace no)
+			(effects
+				(font
+					(size 1.27 1.27)
+				)
+			)
+		)
+		(property "Link" ""
+			(at 358.14 93.98 0)
+			(hide yes)
+			(show_name no)
+			(do_not_autoplace no)
+			(effects
+				(font
+					(size 1.27 1.27)
+				)
+			)
+		)
+		(property "Comp_Name" ""
+			(at 358.14 93.98 0)
+			(show_name no)
+			(do_not_autoplace no)
